File: kicad/ottercontrol.sch (KiCad schematic (older format))
At the start: 79 parts, among them IC1 MAX485, IC2 USBLC6-4, IC3 USBLC6-4, J1 USB_B_Micro, P1 programmer, P2 Conn_01x08, P3 Conn_01x05, P4 Conn_01x02, Q1 Si2367DS, U1 STM32F303CBT6, U2 MAX3051, U6 XL7015, U7 ACT4088, U8 MIC5504-3.3YM5, Y1 16MHz

Commit message: minor cosmetic modifications
Parts:
- R44: MPN (none) -> 103AT
Changed lines of the file:
@@
 EESchema Schematic File Version 4
 LIBS:ottercontrol-cache
-EELAYER 26 0
+EELAYER 29 0
 EELAYER END
 $Descr A4 11693 8268
@@
 F 2 "Resistor_SMD:R_0603_1608Metric" H 6300 6050 50  0001 C CNN
 F 3 "~" H 6300 6050 50  0001 C CNN
-F 4 "" H 6300 7950 50  0001 C CNN "MPN"
+F 4 "103AT" H 6300 7950 50  0001 C CNN "MPN"
 	1    6300 6000
 	1    0    0    -1
